File: owo.kicad_pcb (KiCad board)
At the start: 4 copper layers, 138 parts, among them J1 SJ-43516-SMT-TR, J2 SJ-43516-SMT-TR, J3 5051102291, J4 503398-1892, J5 3.7V, J6 USB4110GFA, Q1 PMOS, Q2 NMOS, SW1 KMR221GLFS, SW2 KMR221GLFS, SW3 KMR221GLFS, SW4 KMR221GLFS, SW5 KMR221GLFS, SW6 KMR221GLFS, SW7 KMR221GLFS, U1 BQ24074RGT, U10 MCP23017_ML, U11 ESP32-C6-WROOM-1, U12 KMR241GLFS, U13 KMR241GLFS, U14 OPA1622, U2 TPS7A20xxxDQN, U3 LM27762, U4 TPS62840DLCR, U5 CD74HC4067M, U6 PCM5122PW, U7 OPA1622, U8 KMR241GLFS, U9 KMR241GLFS, X1 ASE-45.1584MHz, X2 ASE-24.576MHz, Y1 32.768kHz 9pF

Commit message: twt
Routing:
- added copper zone on In1.Cu, net V3.3_SYS
Other:
- copper layers 4 -> 6
Changed lines of the file:
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@@
 		(1 "In1.Cu" signal)
 		(2 "In2.Cu" signal)
+		(3 "In3.Cu" signal)
+		(4 "In4.Cu" signal)
 		(31 "B.Cu" signal)
 		(32 "B.Adhes" user "B.Adhesive")
@@
 			(layer "dielectric 2"
 				(type "core")
-				(thickness 1.24)
+				(thickness 0.535)
 				(material "FR4")
 				(epsilon_r 4.5)
@@
 				(loss_tangent 0.02)
 			)
+			(layer "In3.Cu"
+				(type "copper")
+				(thickness 0.035)
+			)
+			(layer "dielectric 4"
+				(type "core")
+				(thickness 0.535)
+				(material "FR4")
+				(epsilon_r 4.5)
+				(loss_tangent 0.02)
+			)
+			(layer "In4.Cu"
+				(type "copper")
+				(thickness 0.035)
+			)
+			(layer "dielectric 5"
+				(type "prepreg")
+				(thickness 0.1)
+				(material "FR4")
+				(epsilon_r 4.5)
+				(loss_tangent 0.02)
+			)
 			(layer "B.Cu"
 				(type "copper")
@@
 			(outputformat 1)
 			(mirror no)
-			(drillshape 1)
+			(drillshape 0)
 			(scaleselection 1)
 			(outputdirectory "")
@@
 		)
 	)
+	(dimension
+		(type aligned)
+		(layer "B.SilkS")
+		(pts
+			(xy 146.5 98.5) (xy 192.8 98.5)
+		)
+		(height 0)
+		(gr_text "46.3000 mm"
+			(at 169.65 97.4 0)
+			(layer "B.SilkS")
+			(effects
+				(font
+					(size 1 1)
+					(thickness 0.1)
+				)
+				(justify mirror)
+			)
+		)
+		(format
+			(prefix "")
+			(suffix "")
+			(units 3)
+			(units_format 1)
+			(precision 4)
+		)
+		(style
+			(thickness 0.1)
+			(arrow_length 1.27)
+			(text_position_mode 0)
+			(extension_height 0.58642)
+			(extension_offset 0.5) keep_text_aligned)
+	)
+	(dimension
+		(type aligned)
+		(layer "B.SilkS")
+		(pts
+			(xy 140.5 34.4) (xy 140.5 95)
+		)
+		(height 0)
+		(gr_text "60.6000 mm"
+			(at 139.4 64.7 90)
+			(layer "B.SilkS")
+			(effects
+				(font
+					(size 1 1)
+					(thickness 0.1)
+				)
+				(justify mirror)
+			)
+		)
+		(format
+			(prefix "")
+			(suffix "")
+			(units 3)
+			(units_format 1)
+			(precision 4)
+		)
+		(style
+			(thickness 0.1)
+			(arrow_length 1.27)
+			(text_position_mode 0)
+			(extension_height 0.58642)
+			(extension_offset 0.5) keep_text_aligned)
+	)
 	(zone
 		(net 25)
@@
 		(polygon
 			(pts
-				(xy 189.1 70.7) (xy 146.5 70.7) (xy 146.5 75) (xy 182.88449 74.9) (xy 182.9 73.7) (xy 186 73.7)
-				(xy 189.1 73.7) (xy 189.1 73.7)
+				(xy 173.6 70.7) (xy 148.8 70.7) (xy 148.8 75) (xy 173.6 75)
+			)
+		)
+	)
+	(zone
+		(net 3)
+		(net_name "V3.3_SYS")
+		(layer "In1.Cu")
+		(hatch edge 0.5)
+		(priority 5)
+		(connect_pads
+			(clearance 0.5)
+		)
+		(min_thickness 0.25)
+		(filled_areas_thickness no)
+		(fill
+			(thermal_gap 0.5)
+			(thermal_bridge_width 0.5)
+		)
+		(polygon
+			(pts
+				(xy 146.5 94.9) (xy 146.5 89.7) (xy 146.6 89.6) (xy 180.9 89.6) (xy 180.9 62.3) (xy 146.5 62.3)
+				(xy 146.5 34.4) (xy 192.8 34.4) (xy 192.8 94.9)
 			)
 		)
@@
 		(polygon
 			(pts
-				(xy 189.1 76.7) (xy 182.9 76.7) (xy 182.892465 75.5) (xy 146.5 75.5) (xy 146.5 79.7) (xy 189.1 79.7)
+				(xy 173.6 75.5) (xy 148.8 75.5) (xy 148.8 79.8) (xy 173.6 79.8)
 			)
 		)
@@
 		(polygon
 			(pts
-				(xy 146.5 62.6) (xy 146.5 70.3) (xy 146.5 70.3) (xy 189.5 70.3) (xy 189.5 83.8) (xy 189.6 83.9)
-				(xy 192.8 83.9) (xy 192.8 62.6)
+				(xy 146.5 62.6) (xy 146.5 70.3) (xy 146.5 70.3) (xy 174 70.3) (xy 174 80.20056) (xy 148.4 80.229203)
+				(xy 148.4 70.3) (xy 146.5 70.3) (xy 146.5 80.330769) (xy 146.5 89.3) (xy 180.6 89.3) (xy 180.6 62.6)
 			)
 		)
